Commit message: Aug 3 updates

File: legged_examples/legged_unitree/legged_unitree_description/urdf/husky_defined1.xacro (robot description, xacro)
@@ -7,6 +7,12 @@
   <xacro:property name="free_joint_sfriction" value="0" />
   <xacro:property name="efflim" value="33.5" />
-  <xacro:property name="r_axis" value="1" />
-  <xacro:property name="l_axis" value="1" />
+  <xacro:property name="r_hip_frontal_ipos" value="0.0440" />
+  <xacro:property name="l_hip_frontal_ipos" value="3.0976" />
+  <xacro:property name="l_hip_frontal_lowlim" value="-0.1745" />
+  <xacro:property name="l_hip_frontal_uplim" value="1.3963" />
+  <xacro:property name="r_hip_frontal_lowlim" value="-1.3963" />
+  <xacro:property name="r_hip_frontal_uplim" value="0.1745" />
+  <xacro:property name="r_axis" value="-1" />
+  <xacro:property name="l_axis" value="-1" />
   <gazebo>
   <plugin filename="liblegged_hw_sim.so" name="gazebo_ros_control">
@@ -52,8 +58,4 @@
     <disableFixedJointLumping>true</disableFixedJointLumping>
   </gazebo>
-  <xacro:property name="r_hip_frontal_ipos" value="-0.1745" />
-  <xacro:property name="l_hip_frontal_ipos" value="-2.9671" />
-  <xacro:property name="l_hip_frontal_lowlim" value="-0.5236" />
-  <xacro:property name="l_hip_frontal_uplim" value="0.5236" />
   <joint name="RF_HAA" type="revolute">
     <parent link="base"/>
@@ -62,5 +64,5 @@
     <axis xyz="0.0 0.0 1.0" />
     <dynamics damping="${motor_damping}" friction="${motor_sfriction}"/>
-    <limit effort="${efflim}" lower="${l_hip_frontal_lowlim}" upper="${l_hip_frontal_uplim}" velocity="8.7267"/>
+    <limit effort="${efflim}" lower="${r_hip_frontal_lowlim}" upper="${r_hip_frontal_uplim}" velocity="8.7267"/>
   </joint>
   <joint name="LF_HAA" type="revolute">
@@ -86,10 +88,12 @@
     <axis xyz="0 0 1" />
     <dynamics damping="${motor_damping}" friction="${motor_sfriction}"/>
-    <limit effort="${efflim}" lower="${l_hip_frontal_lowlim}" upper="${l_hip_frontal_uplim}" velocity="8.7267"/>
-  </joint>
-  <xacro:property name="l_hip_sagittal_ipos" value="-1.0472" />
-  <xacro:property name="r_hip_sagittal_ipos" value="-2.0944" />
-  <xacro:property name="l_hip_sagittal_lowlim" value="-0.8727" />
-  <xacro:property name="l_hip_sagittal_uplim" value="0.8727" />
+    <limit effort="${efflim}" lower="${r_hip_frontal_lowlim}" upper="${r_hip_frontal_uplim}" velocity="8.7267"/>
+  </joint>
+  <xacro:property name="l_hip_sagittal_ipos" value="-0.8496" />
+  <xacro:property name="r_hip_sagittal_ipos" value="-2.2920" />
+  <xacro:property name="l_hip_sagittal_lowlim" value="-0.7212" />
+  <xacro:property name="l_hip_sagittal_uplim" value="0.8496" />
+  <xacro:property name="r_hip_sagittal_lowlim" value="-0.8496" />
+  <xacro:property name="r_hip_sagittal_uplim" value="0.7212" />
   <joint name="RF_HFE" type="revolute">
     <parent link="RF_hip"/>
@@ -98,5 +102,5 @@
     <axis xyz="0.0 0 ${r_axis}" />
     <dynamics damping="${motor_damping}" friction="${motor_sfriction}"/>
-    <limit effort="${efflim}" lower="${l_hip_sagittal_lowlim}" upper="${l_hip_sagittal_uplim}" velocity="8.7267"/>
+    <limit effort="${efflim}" lower="${r_hip_sagittal_lowlim}" upper="${r_hip_sagittal_uplim}" velocity="8.7267"/>
   </joint>
   <joint name="LF_HFE" type="revolute">
@@ -122,10 +126,12 @@
     <axis xyz="0.0 0 ${r_axis}" />
     <dynamics damping="${motor_damping}" friction="${motor_sfriction}"/>
-    <limit effort="${efflim}" lower="${l_hip_sagittal_lowlim}" upper="${l_hip_sagittal_uplim}" velocity="8.7267"/>
-  </joint>
-  <xacro:property name="l_knee_ipos" value="1.6755" />
-  <xacro:property name="r_knee_ipos" value="-1.6755" />
-  <xacro:property name="l_knee_lowlim" value="-0.6981" />
-  <xacro:property name="l_knee_uplim" value="0.6981" />
+    <limit effort="${efflim}" lower="${r_hip_sagittal_lowlim}" upper="${r_hip_sagittal_uplim}" velocity="8.7267"/>
+  </joint>
+  <xacro:property name="l_knee_ipos" value="1.6813" />
+  <xacro:property name="r_knee_ipos" value="-1.6813" />
+  <xacro:property name="l_knee_lowlim" value="-0.8331" />
+  <xacro:property name="l_knee_uplim" value="0.73" />
+  <xacro:property name="r_knee_lowlim" value="-0.73" />
+  <xacro:property name="r_knee_uplim" value="0.8331" />
   <joint name="RF_KFE" type="revolute">
     <parent link="RF_thigh"/>
@@ -134,5 +140,5 @@
     <axis xyz="0.0 0.0 ${r_axis}" />
     <dynamics damping="${motor_damping}" friction="${motor_sfriction}"/>
-    <limit effort="${efflim}" lower="${l_knee_lowlim}" upper="${l_knee_uplim}" velocity="8.7267"/>
+    <limit effort="${efflim}" lower="${r_knee_lowlim}" upper="${r_knee_uplim}" velocity="8.7267"/>
   </joint>
   <joint name="LF_KFE" type="revolute">
@@ -158,5 +164,5 @@
     <axis xyz="0.0 0.0 ${r_axis}" />
     <dynamics damping="${motor_damping}" friction="${motor_sfriction}"/>
-    <limit effort="${efflim}" lower="${l_knee_lowlim}" upper="${l_knee_uplim}" velocity="8.7267"/>
+    <limit effort="${efflim}" lower="${r_knee_lowlim}" upper="${r_knee_uplim}" velocity="8.7267"/>
   </joint>
   <!--ANKLES-->

File: legged_examples/legged_unitree/legged_unitree_description/urdf/husky_error4.xacro (robot description, xacro)
@@ -13,6 +13,6 @@
   <xacro:property name="r_hip_frontal_lowlim" value="-1.3963" />
   <xacro:property name="r_hip_frontal_uplim" value="0.1745" />
-  <xacro:property name="r_axis" value="-1" />
-  <xacro:property name="l_axis" value="-1" />
+  <xacro:property name="r_axis" value="1" />
+  <xacro:property name="l_axis" value="1" />
   <gazebo>
   <plugin filename="liblegged_hw_sim.so" name="gazebo_ros_control">

File: legged_examples/legged_unitree/legged_unitree_description/urdf/husky_error5.xacro (robot description, xacro)
@@ -7,6 +7,12 @@
   <xacro:property name="free_joint_sfriction" value="0" />
   <xacro:property name="efflim" value="33.5" />
-  <xacro:property name="r_axis" value="1" />
-  <xacro:property name="l_axis" value="1" />
+  <xacro:property name="r_hip_frontal_ipos" value="0.0440" />
+  <xacro:property name="l_hip_frontal_ipos" value="3.0976" />
+  <xacro:property name="l_hip_frontal_lowlim" value="-0.1745" />
+  <xacro:property name="l_hip_frontal_uplim" value="1.3963" />
+  <xacro:property name="r_hip_frontal_lowlim" value="-1.3963" />
+  <xacro:property name="r_hip_frontal_uplim" value="0.1745" />
+  <xacro:property name="r_axis" value="-1" />
+  <xacro:property name="l_axis" value="-1" />
   <gazebo>
   <plugin filename="liblegged_hw_sim.so" name="gazebo_ros_control">
@@ -52,8 +58,4 @@
     <disableFixedJointLumping>true</disableFixedJointLumping>
   </gazebo>
-  <xacro:property name="r_hip_frontal_ipos" value="-0.1745" />
-  <xacro:property name="l_hip_frontal_ipos" value="-2.9671" />
-  <xacro:property name="l_hip_frontal_lowlim" value="-0.5236" />
-  <xacro:property name="l_hip_frontal_uplim" value="0.5236" />
   <joint name="RF_HAA" type="revolute">
     <parent link="base"/>
@@ -62,5 +64,5 @@
     <axis xyz="0.0 0.0 1.0" />
     <dynamics damping="${motor_damping}" friction="${motor_sfriction}"/>
-    <limit effort="${efflim}" lower="${l_hip_frontal_lowlim}" upper="${l_hip_frontal_uplim}" velocity="8.7267"/>
+    <limit effort="${efflim}" lower="${r_hip_frontal_lowlim}" upper="${r_hip_frontal_uplim}" velocity="8.7267"/>
   </joint>
   <joint name="LF_HAA" type="revolute">
@@ -86,10 +88,12 @@
     <axis xyz="0 0 1" />
     <dynamics damping="${motor_damping}" friction="${motor_sfriction}"/>
-    <limit effort="${efflim}" lower="${l_hip_frontal_lowlim}" upper="${l_hip_frontal_uplim}" velocity="8.7267"/>
-  </joint>
-  <xacro:property name="l_hip_sagittal_ipos" value="-1.0472" />
-  <xacro:property name="r_hip_sagittal_ipos" value="-2.0944" />
-  <xacro:property name="l_hip_sagittal_lowlim" value="-0.8727" />
-  <xacro:property name="l_hip_sagittal_uplim" value="0.8727" />
+    <limit effort="${efflim}" lower="${r_hip_frontal_lowlim}" upper="${r_hip_frontal_uplim}" velocity="8.7267"/>
+  </joint>
+  <xacro:property name="l_hip_sagittal_ipos" value="-0.8496" />
+  <xacro:property name="r_hip_sagittal_ipos" value="-2.2920" />
+  <xacro:property name="l_hip_sagittal_lowlim" value="-0.7212" />
+  <xacro:property name="l_hip_sagittal_uplim" value="0.8496" />
+  <xacro:property name="r_hip_sagittal_lowlim" value="-0.8496" />
+  <xacro:property name="r_hip_sagittal_uplim" value="0.7212" />
   <joint name="RF_HFE" type="revolute">
     <parent link="RF_hip"/>
@@ -98,5 +102,5 @@
     <axis xyz="0.0 0 ${r_axis}" />
     <dynamics damping="${motor_damping}" friction="${motor_sfriction}"/>
-    <limit effort="${efflim}" lower="${l_hip_sagittal_lowlim}" upper="${l_hip_sagittal_uplim}" velocity="8.7267"/>
+    <limit effort="${efflim}" lower="${r_hip_sagittal_lowlim}" upper="${r_hip_sagittal_uplim}" velocity="8.7267"/>
   </joint>
   <joint name="LF_HFE" type="revolute">
@@ -122,10 +126,12 @@
     <axis xyz="0.0 0 ${r_axis}" />
     <dynamics damping="${motor_damping}" friction="${motor_sfriction}"/>
-    <limit effort="${efflim}" lower="${l_hip_sagittal_lowlim}" upper="${l_hip_sagittal_uplim}" velocity="8.7267"/>
-  </joint>
-  <xacro:property name="l_knee_ipos" value="1.6755" />
-  <xacro:property name="r_knee_ipos" value="-1.6755" />
-  <xacro:property name="l_knee_lowlim" value="-0.6981" />
-  <xacro:property name="l_knee_uplim" value="0.6981" />
+    <limit effort="${efflim}" lower="${r_hip_sagittal_lowlim}" upper="${r_hip_sagittal_uplim}" velocity="8.7267"/>
+  </joint>
+  <xacro:property name="l_knee_ipos" value="1.6813" />
+  <xacro:property name="r_knee_ipos" value="-1.6813" />
+  <xacro:property name="l_knee_lowlim" value="-0.8331" />
+  <xacro:property name="l_knee_uplim" value="0.73" />
+  <xacro:property name="r_knee_lowlim" value="-0.73" />
+  <xacro:property name="r_knee_uplim" value="0.8331" />
   <joint name="RF_KFE" type="revolute">
     <parent link="RF_thigh"/>
@@ -134,5 +140,5 @@
     <axis xyz="0.0 0.0 ${r_axis}" />
     <dynamics damping="${motor_damping}" friction="${motor_sfriction}"/>
-    <limit effort="${efflim}" lower="${l_knee_lowlim}" upper="${l_knee_uplim}" velocity="8.7267"/>
+    <limit effort="${efflim}" lower="${r_knee_lowlim}" upper="${r_knee_uplim}" velocity="8.7267"/>
   </joint>
   <joint name="LF_KFE" type="revolute">
@@ -158,13 +164,11 @@
     <axis xyz="0.0 0.0 ${r_axis}" />
     <dynamics damping="${motor_damping}" friction="${motor_sfriction}"/>
-    <limit effort="${efflim}" lower="${l_knee_lowlim}" upper="${l_knee_uplim}" velocity="8.7267"/>
-  </joint>
-  <!--ANKLES-->
+    <limit effort="${efflim}" lower="${r_knee_lowlim}" upper="${r_knee_uplim}" velocity="8.7267"/>
+  </joint>
+  <!--ANKLES (MADE FIXED FOR ONE-TO-ONE)-->
   <xacro:property name="l_ankle_lowlim" value="-0.65" />
   <xacro:property name="l_ankle_uplim" value="0.92" />
   <xacro:property name="r_ankle_lowlim" value="-0.92" />
   <xacro:property name="r_ankle_uplim" value="0.65" />
-  <!--REAL FOOT SECTION 1/3 (COMMENT THIS IN, COMMENT BELOW OUT)-->
-  <!--
   <joint name="RF_ankle" type="revolute">
     <parent link="RF_calf"/>
@@ -199,4 +203,5 @@
     <limit effort="${efflim}" lower="${r_ankle_lowlim}" upper="${r_ankle_uplim}" velocity="8.7267"/>
   </joint>
+  <!--foot nub-->
   <joint name="RF_foot_fixed" type="fixed">
     <parent link="RF_fut"/>
@@ -219,29 +224,4 @@
     <origin rpy="0 0 0"   xyz="0.0 0.0 0.0"/>
   </joint>
-  -->
-  <!--REAL FOOT SECTION END-->
-  <!--NUB FOOT SECTION (COMMENT THIS IN, COMMENT ABOVE OUT)-->
-  <joint name="RF_foot_fixed" type="fixed">
-    <parent link="RF_calf"/>
-    <child link="RF_FOOT"/>
-    <origin rpy="0 0 0"   xyz="0.0 0.0 0.0"/>
-  </joint>
-  <joint name="LF_foot_fixed" type="fixed">
-    <parent link="LF_calf"/>
-    <child link="LF_FOOT"/>
-    <origin rpy="0 0 0"   xyz="0.0 0.0 0.0"/>
-  </joint>
-  <joint name="LH_foot_fixed" type="fixed">
-    <parent link="LH_calf"/>
-    <child link="LH_FOOT"/>
-    <origin rpy="0 0 0"   xyz="0.0 0.0 0.0"/>
-  </joint>
-  <joint name="RH_foot_fixed" type="fixed">
-    <parent link="RH_calf"/>
-    <child link="RH_FOOT"/>
-    <origin rpy="0 0 0"   xyz="0.0 0.0 0.0"/>
-  </joint>
-  -->
-  <!--NUB FOOT SECTION END-->
   <gazebo reference="RF_foot_fixed">
     <disableFixedJointLumping>true</disableFixedJointLumping>
@@ -679,6 +659,4 @@
     <self_collide>1</self_collide>
   </gazebo>
-  <!--REAL FOOT SECTION 2/3 (COMMENT THIS IN, COMMENT BELOW OUT)-->
-  <!--
   <xacro:property name="foot_ix" value="0.01" />
   <xacro:property name="foot_length" value="0.16" />
@@ -794,13 +772,4 @@
     <self_collide>1</self_collide>
   </gazebo>
-  -->
-  <!--REAL FOOT SECTION END-->
-  <!--NUB FOOT SECTION (COMMENT THIS IN, COMMENT ABOVE OUT)-->
-  <xacro:property name="foot_ix" value="0.01" />
-  <xacro:property name="foot_length" value="0.16" />
-  <xacro:property name="foot_radius" value="0.01" />
-  <xacro:property name="foot_sphere_ix" value="0.342" />
-  <xacro:property name="foot_sphere_radius" value="0.02" />
-  <!--NUB FOOT SECTION END-->
   <link name="RF_FOOT">
     <inertial>
@@ -883,5 +852,4 @@
     <kd value="100.0"/>
   </gazebo>
-  <!--CONTROL ROD SECTION 1/2-->
   <!--
   <joint name="fr_control_rod" type="revolute">
@@ -1006,5 +974,4 @@
   </link>
   -->
-  <!--CONTROL ROD SECTION END-->
   <transmission name="RF_HAA_trans">
     <type>transmission_interface/SimpleTransmission</type>
@@ -1127,6 +1094,4 @@
     </actuator>
   </transmission>
-  <!--REAL FOOT SECTION 3/3 (COMMENT THIS IN, NO NEED TO COMMENT OUT)-->
-  <!--
   <transmission name="RF_ankle_trans">
     <type>transmission_interface/SimpleTransmission</type>
@@ -1169,7 +1134,4 @@
     </actuator>
   </transmission>
-  -->
-  <!--REAL FOOT SECTION END-->
-  <!--CONTROL ROD SECTION 2/2-->
   <!--
   <transmission name="fr_rod_joint_trans">
@@ -1214,5 +1176,4 @@
   </transmission>
   -->
-  <!--CONTROL ROD SECTION END-->
   <gazebo>
   <plugin name="RF_foot_fixed_mimic" filename="libroboticsgroup_gazebo_mimic_joint_plugin.so">
@@ -1256,4 +1217,5 @@
     <robotNamespace>/</robotNamespace>
   </plugin>
+<!--
   <plugin name="fr_control_rod_mimic" filename="libroboticsgroup_gazebo_mimic_joint_plugin.so">
     <joint>RF_KFE</joint>
@@ -1296,4 +1258,5 @@
     <robotNamespace>/</robotNamespace>
   </plugin>
+  -->
   </gazebo>
 </robot>
