Commit message: ardupilot

File: husky_description/urdf/tmp.urdf (robot description, URDF)
Before this commit: robot husky, 31 links, 30 joints
Links:
- removed link fake_front_left_blade
- removed link fake_front_right_blade
- removed link fake_rear_left_blade
- removed link fake_rear_right_blade
- added link front_left_blade, mass 0.0061028301426362
- added link front_right_blade, mass 0.00610290216434297
- added link rear_left_blade, mass 0.00610274937825579
- added link rear_right_blade, mass 0.00610270077025495
- link LF_FOOT: geometry collision sphere radius=0.02
- link LF_calf: geometry collision cylinder length=0.32 radius=0.01; visual mesh filename=package://husky_description/meshes/fr_tibia.STL scale=1 1 1
- link LF_fut: geometry collision cylinder length=0.16 radius=0.01; visual mesh filename=package://husky_description/meshes/fr_foot.STL scale=1 1 1
- link LF_hip: geometry collision cylinder length=0.08 radius=0.03; visual mesh filename=package://husky_description/meshes/bl_hip.STL scale=1 1 1
- link LF_thigh: geometry collision cylinder length=0.05 radius=0.03; collision cylinder length=0.06 radius=0.03
- link LH_FOOT: geometry collision sphere radius=0.02
- link LH_calf: geometry collision cylinder length=0.32 radius=0.01; visual mesh filename=package://husky_description/meshes/fr_tibia.STL scale=1 1 1
- link LH_fut: geometry collision cylinder length=0.16 radius=0.01; visual mesh filename=package://husky_description/meshes/fr_foot.STL scale=1 1 1
- link LH_hip: geometry collision cylinder length=0.08 radius=0.03; visual mesh filename=package://husky_description/meshes/bl_hip.STL scale=1 1 1
- link LH_thigh: geometry collision cylinder length=0.05 radius=0.03; collision cylinder length=0.06 radius=0.03
- link RF_FOOT: geometry collision sphere radius=0.02
- link RF_calf: geometry collision cylinder length=0.32 radius=0.01; visual mesh filename=package://husky_description/meshes/fr_tibia.STL scale=1 1 1
- link RF_fut: geometry collision cylinder length=0.16 radius=0.01; visual mesh filename=package://husky_description/meshes/fr_foot.STL scale=1 1 1
- link RF_hip: geometry collision cylinder length=0.08 radius=0.03; visual mesh filename=package://husky_description/meshes/fr_hip.STL scale=1 1 1
- link RF_thigh: geometry collision cylinder length=0.05 radius=0.03; collision cylinder length=0.06 radius=0.03
- link RH_FOOT: geometry collision sphere radius=0.02
- link RH_calf: geometry collision cylinder length=0.32 radius=0.01; visual mesh filename=package://husky_description/meshes/fr_tibia.STL scale=1 1 1
- link RH_fut: geometry collision cylinder length=0.16 radius=0.01; visual mesh filename=package://husky_description/meshes/fr_foot.STL scale=1 1 1
- link RH_hip: geometry collision cylinder length=0.08 radius=0.03; visual mesh filename=package://husky_description/meshes/fr_hip.STL scale=1 1 1
- link RH_thigh: geometry collision cylinder length=0.05 radius=0.03; collision cylinder length=0.06 radius=0.03
- link base: geometry collision box size=0.3 0.1 0.12; collision box size=0.3 0.1 0.28
- link bl_fibula: geometry collision cylinder length=0.24 radius=0.01; visual mesh filename=package://husky_description/meshes/fr_fibula.STL scale=1 1 1
- link br_fibula: geometry collision cylinder length=0.24 radius=0.01; visual mesh filename=package://husky_description/meshes/fr_fibula.STL scale=1 1 1
- link fl_fibula: geometry collision cylinder length=0.24 radius=0.01; visual mesh filename=package://husky_description/meshes/fr_fibula.STL scale=1 1 1
- link fr_fibula: geometry collision cylinder length=0.24 radius=0.01; visual mesh filename=package://husky_description/meshes/fr_fibula.STL scale=1 1 1
Joints:
- removed joint fake_front_left_blade_joint
- removed joint fake_front_right_blade_joint
- removed joint fake_rear_left_blade_joint
- removed joint fake_rear_right_blade_joint
- added joint front_left_blade_joint: type revolute, parent base, child front_left_blade, origin xyz=0 0.162 0.062522 rpy=0 0 0, axis 0 0 1, limit lower=-1e+16 upper=1e+16 effort=10000 velocity=10000
- added joint front_right_blade_joint: type revolute, parent base, child front_right_blade, origin xyz=0 0.162 -0.065427 rpy=-3.1416 0 -0.0052077, axis 0 0 1, limit lower=-1e+16 upper=1e+16 effort=10000 velocity=10000
- added joint rear_left_blade_joint: type revolute, parent base, child rear_left_blade, origin xyz=0 0.162 0.061129 rpy=-0.0099006 0 0.018227, axis 0 -0.0099004 0.99995, limit lower=-1e+16 upper=1e+16 effort=10000 velocity=10000
- added joint rear_right_blade_joint: type revolute, parent base, child rear_right_blade, origin xyz=0 0.162 -0.065431 rpy=3.1416 0 0, axis 0 0 1, limit lower=-1e+16 upper=1e+16 effort=10000 velocity=10000
- joint LF_HAA: limit lower=${l_hip_frontal_lowlim} upper=${l_hip_frontal_uplim} effort=${efflim} velocity=8.7267 -> lower=0 upper=0.08726646259971647 effort=33.5 velocity=8.7267; origin xyz=0.2087 0.045 0.0001 rpy=-1.5708 ${l_hip_frontal_ipos} -1.5708 -> xyz=0.2087 0.045 0.0001 rpy=-1.5708 -2.9670597283903604 -1.5708
- joint LF_HFE: axis 0 0.0 ${l_axis} -> 0 0.0 1; limit lower=${fl_hip_sagittal_lowlim} upper=${fl_hip_sagittal_uplim} effort=${efflim} velocity=8.7267 -> lower=0 upper=0.20943951023931953 effort=33.5 velocity=8.7267; origin xyz=0.1031 0.0 0.0 rpy=-1.5708 ${fl_hip_sagittal_ipos} -1.5708 -> xyz=0.1031 0.0 0.0 rpy=-1.5708 -1.019097750239489 -1.5708
- joint LF_KFE: axis 0.0 0.0 ${l_axis} -> 0.0 0.0 1; limit lower=${l_knee_lowlim} upper=${l_knee_uplim} effort=${efflim} velocity=8.7267 -> lower=-1.0471975511965976 upper=0 effort=33.5 velocity=8.7267; origin xyz=0.18 0.0 -0.0431 rpy=0 0 ${l_knee_ipos} -> xyz=0.18 0.0 -0.0431 rpy=0 0 2.4113468945553653
- joint LF_ankle: limit lower=${l_ankle_lowlim} upper=${l_ankle_uplim} effort=${efflim} velocity=8.7267 -> lower=-1.5707963267948966 upper=1.5707963267948966 effort=33.5 velocity=8.7267; origin xyz=0.333 0.0 0.0 rpy=0 0 ${r_knee_ipos} -> xyz=0.333 0.0 0.0 rpy=0 0 -2.4113468945553653
- joint LH_HAA: limit lower=${l_hip_frontal_lowlim} upper=${l_hip_frontal_uplim} effort=${efflim} velocity=8.7267 -> lower=0 upper=0.08726646259971647 effort=33.5 velocity=8.7267; origin xyz=-0.1862 0.045 0.0002 rpy=-1.5708 ${l_hip_frontal_ipos} -1.5708 -> xyz=-0.1862 0.045 0.0002 rpy=-1.5708 -2.9670597283903604 -1.5708
- joint LH_HFE: axis 0.0 0.0 ${l_axis} -> 0.0 0.0 1; limit lower=${bl_hip_sagittal_lowlim} upper=${bl_hip_sagittal_uplim} effort=${efflim} velocity=8.7267 -> lower=0 upper=0.20943951023931953 effort=33.5 velocity=8.7267; origin xyz=0.1031 0.0 0.0 rpy=-1.5708 ${bl_hip_sagittal_ipos} -1.5708 -> xyz=0.1031 0.0 0.0 rpy=-1.5708 -0.8496262798708396 -1.5708
- joint LH_KFE: axis 0.0 0.0 ${l_axis} -> 0.0 0.0 1; limit lower=${l_knee_lowlim} upper=${l_knee_uplim} effort=${efflim} velocity=8.7267 -> lower=-1.0471975511965976 upper=0 effort=33.5 velocity=8.7267; origin xyz=0.18 0.0 -0.0431 rpy=0 0 ${l_knee_ipos} -> xyz=0.18 0.0 -0.0431 rpy=0 0 2.4113468945553653
- joint LH_ankle: limit lower=${l_ankle_lowlim} upper=${l_ankle_uplim} effort=${efflim} velocity=8.7267 -> lower=-1.5707963267948966 upper=1.5707963267948966 effort=33.5 velocity=8.7267; origin xyz=0.333 0.0 0.0 rpy=0 0 ${r_knee_ipos} -> xyz=0.333 0.0 0.0 rpy=0 0 -2.4113468945553653
- joint RF_HAA: limit lower=${r_hip_frontal_lowlim} upper=${r_hip_frontal_uplim} effort=${efflim} velocity=8.7267 -> lower=-0.08726646259971647 upper=0 effort=33.5 velocity=8.7267; origin xyz=0.2087 -0.045 0.0001 rpy=-1.5708 ${r_hip_frontal_ipos} -1.5708 -> xyz=0.2087 -0.045 0.0001 rpy=-1.5708 -0.17453292519943295 -1.5708
- joint RF_HFE: axis 0.0 0 ${r_axis} -> 0.0 0 1; limit lower=${fr_hip_sagittal_lowlim} upper=${fr_hip_sagittal_uplim} effort=${efflim} velocity=8.7267 -> lower=-0.20943951023931953 upper=0 effort=33.5 velocity=8.7267; origin xyz=0.1031 0.0 0.0 rpy=-1.5708 ${fr_hip_sagittal_ipos} -1.5708 -> xyz=0.1031 0.0 0.0 rpy=-1.5708 -2.122494903350304 -1.5708
- joint RF_KFE: axis 0.0 0.0 ${r_axis} -> 0.0 0.0 1; limit lower=${r_knee_lowlim} upper=${r_knee_uplim} effort=${efflim} velocity=8.7267 -> lower=0 upper=1.0471975511965976 effort=33.5 velocity=8.7267; origin xyz=0.18 0.0 -0.0431 rpy=0 0 ${r_knee_ipos} -> xyz=0.18 0.0 -0.0431 rpy=0 0 -2.4113468945553653
- joint RF_ankle: limit lower=${r_ankle_lowlim} upper=${r_ankle_uplim} effort=${efflim} velocity=8.7267 -> lower=-1.5707963267948966 upper=1.5707963267948966 effort=33.5 velocity=8.7267; origin xyz=0.333 0.0 0.0 rpy=0 0 ${l_knee_ipos} -> xyz=0.333 0.0 0.0 rpy=0 0 2.4113468945553653
- joint RH_HAA: limit lower=${r_hip_frontal_lowlim} upper=${r_hip_frontal_uplim} effort=${efflim} velocity=8.7267 -> lower=-0.08726646259971647 upper=0 effort=33.5 velocity=8.7267; origin xyz=-0.1862 -0.045 0.0002 rpy=-1.5708 ${r_hip_frontal_ipos} -1.5708 -> xyz=-0.1862 -0.045 0.0002 rpy=-1.5708 -0.17453292519943295 -1.5708
- joint RH_HFE: axis 0.0 0 ${r_axis} -> 0.0 0 1; limit lower=${br_hip_sagittal_lowlim} upper=${br_hip_sagittal_uplim} effort=${efflim} velocity=8.7267 -> lower=-0.20943951023931953 upper=0 effort=33.5 velocity=8.7267; origin xyz=0.1031 0.0 0.0 rpy=-1.5708 ${br_hip_sagittal_ipos} -1.5708 -> xyz=0.1031 0.0 0.0 rpy=-1.5708 -2.2919663737189535 -1.5708
- joint RH_KFE: axis 0.0 0.0 ${r_axis} -> 0.0 0.0 1; limit lower=${r_knee_lowlim} upper=${r_knee_uplim} effort=${efflim} velocity=8.7267 -> lower=0 upper=1.0471975511965976 effort=33.5 velocity=8.7267; origin xyz=0.18 0.0 -0.0431 rpy=0 0 ${r_knee_ipos} -> xyz=0.18 0.0 -0.0431 rpy=0 0 -2.4113468945553653
- joint RH_ankle: limit lower=${r_ankle_lowlim} upper=${r_ankle_uplim} effort=${efflim} velocity=8.7267 -> lower=-1.5707963267948966 upper=1.5707963267948966 effort=33.5 velocity=8.7267; origin xyz=0.333 0.0 0.0 rpy=0 0 ${l_knee_ipos} -> xyz=0.333 0.0 0.0 rpy=0 0 2.4113468945553653
- joint bl_control_rod: limit lower=${l_knee_lowlim} upper=${l_knee_uplim} effort=${efflim} velocity=8.7267 -> lower=-1.0471975511965976 upper=0 effort=33.5 velocity=8.7267; origin xyz=0.12 0.0 -0.0431 rpy=0 0.0 ${l_knee_ipos} -> xyz=0.12 0.0 -0.0431 rpy=0 0.0 2.4113468945553653
- joint br_control_rod: limit lower=${r_knee_lowlim} upper=${r_knee_uplim} effort=${efflim} velocity=8.7267 -> lower=0 upper=1.0471975511965976 effort=33.5 velocity=8.7267; origin xyz=0.12 0.0 -0.0431 rpy=0 0.0 ${r_knee_ipos} -> xyz=0.12 0.0 -0.0431 rpy=0 0.0 -2.4113468945553653
- joint fl_control_rod: limit lower=${l_knee_lowlim} upper=${l_knee_uplim} effort=${efflim} velocity=8.7267 -> lower=-1.0471975511965976 upper=0 effort=33.5 velocity=8.7267; origin xyz=0.12 0.0 -0.0431 rpy=0 0.0 ${l_knee_ipos} -> xyz=0.12 0.0 -0.0431 rpy=0 0.0 2.4113468945553653
- joint fr_control_rod: limit lower=${r_knee_lowlim} upper=${r_knee_uplim} effort=${efflim} velocity=8.7267 -> lower=0 upper=1.0471975511965976 effort=33.5 velocity=8.7267; origin xyz=0.12 0.0 -0.0431 rpy=0 0.0 ${r_knee_ipos} -> xyz=0.12 0.0 -0.0431 rpy=0 0.0 -2.4113468945553653
