Commit message: updated inertias

File: husky_description/urdf/husky.xacro (robot description, xacro)
@@ -260,5 +260,5 @@
     <inertial>
       <mass value="3.1895"/>
-      <origin rpy="0.0 0.0 -1.5708" xyz="0.0001 0.0301 0.0241"/>
+      <origin rpy="0.0 0.0 -1.5708" xyz="0.0301 -0.0001 0.0241"/>
       <inertia ixx="0.0170990623" ixy="3.09e-08" ixz="-5.394e-07" iyy="0.0115476717" iyz="4.77948e-05" izz="0.0268461573"/>
     </inertial>
@@ -285,5 +285,5 @@
     <inertial>
       <mass value="0.0431"/>
-      <origin rpy="3.1416 0.0 0.0" xyz="0.0236 -0.0001 -0.003"/>
+      <origin rpy="3.1416 0.0 0.0" xyz="0.0236 0.0001 0.003"/>
       <inertia ixx="9.9689e-06" ixy="7.49e-08" ixz="-2.3932e-06" iyy="2.49545e-05" iyz="5.1e-09" izz="2.81284e-05"/>
     </inertial>
@@ -307,5 +307,5 @@
     <inertial>
       <mass value="0.0431"/>
-      <origin rpy="3.1416 0.0 0.0" xyz="0.0236 -0.0001 -0.003"/>
+      <origin rpy="3.1416 0.0 0.0" xyz="0.0236 0.0001 0.003"/>
       <inertia ixx="9.9689e-06" ixy="7.49e-08" ixz="-2.3932e-06" iyy="2.49545e-05" iyz="5.1e-09" izz="2.81284e-05"/>
     </inertial>
@@ -329,5 +329,5 @@
     <inertial>
       <mass value="0.0431"/>
-      <origin rpy="3.1416 0.0 0.0" xyz="0.0236 -0.0001 -0.003"/>
+      <origin rpy="3.1416 0.0 0.0" xyz="0.0236 0.0001 0.003"/>
       <inertia ixx="9.9689e-06" ixy="7.49e-08" ixz="-2.3932e-06" iyy="2.49545e-05" iyz="5.1e-09" izz="2.81284e-05"/>
     </inertial>
@@ -351,5 +351,5 @@
     <inertial>
       <mass value="0.0431"/>
-      <origin rpy="3.1416 0.0 0.0" xyz="0.0236 -0.0001 -0.003"/>
+      <origin rpy="3.1416 0.0 0.0" xyz="0.0236 0.0001 0.003"/>
       <inertia ixx="9.9689e-06" ixy="7.49e-08" ixz="-2.3932e-06" iyy="2.49545e-05" iyz="5.1e-09" izz="2.81284e-05"/>
     </inertial>

File: husky_description/urdf/husky_defined1.xacro (robot description, xacro)
@@ -266,5 +266,5 @@
     <inertial>
       <mass value="3.1895"/>
-      <origin rpy="0.0 0.0 -1.5708" xyz="0.0001 0.0301 0.0241"/>
+      <origin rpy="0.0 0.0 -1.5708" xyz="0.0301 -0.0001 0.0241"/>
       <inertia ixx="0.0170990623" ixy="3.09e-08" ixz="-5.394e-07" iyy="0.0115476717" iyz="4.77948e-05" izz="0.0268461573"/>
     </inertial>
@@ -291,5 +291,5 @@
     <inertial>
       <mass value="0.0431"/>
-      <origin rpy="3.1416 0.0 0.0" xyz="0.0236 -0.0001 -0.003"/>
+      <origin rpy="3.1416 0.0 0.0" xyz="0.0236 0.0001 0.003"/>
       <inertia ixx="9.9689e-06" ixy="7.49e-08" ixz="-2.3932e-06" iyy="2.49545e-05" iyz="5.1e-09" izz="2.81284e-05"/>
     </inertial>
@@ -313,5 +313,5 @@
     <inertial>
       <mass value="0.0431"/>
-      <origin rpy="3.1416 0.0 0.0" xyz="0.0236 -0.0001 -0.003"/>
+      <origin rpy="3.1416 0.0 0.0" xyz="0.0236 0.0001 0.003"/>
       <inertia ixx="9.9689e-06" ixy="7.49e-08" ixz="-2.3932e-06" iyy="2.49545e-05" iyz="5.1e-09" izz="2.81284e-05"/>
     </inertial>
@@ -335,5 +335,5 @@
     <inertial>
       <mass value="0.0431"/>
-      <origin rpy="3.1416 0.0 0.0" xyz="0.0236 -0.0001 -0.003"/>
+      <origin rpy="3.1416 0.0 0.0" xyz="0.0236 0.0001 0.003"/>
       <inertia ixx="9.9689e-06" ixy="7.49e-08" ixz="-2.3932e-06" iyy="2.49545e-05" iyz="5.1e-09" izz="2.81284e-05"/>
     </inertial>
@@ -357,5 +357,5 @@
     <inertial>
       <mass value="0.0431"/>
-      <origin rpy="3.1416 0.0 0.0" xyz="0.0236 -0.0001 -0.003"/>
+      <origin rpy="3.1416 0.0 0.0" xyz="0.0236 0.0001 0.003"/>
       <inertia ixx="9.9689e-06" ixy="7.49e-08" ixz="-2.3932e-06" iyy="2.49545e-05" iyz="5.1e-09" izz="2.81284e-05"/>
     </inertial>

File: husky_description/urdf/husky_hobbler.xacro (robot description, xacro)
@@ -208,5 +208,5 @@
     <inertial>
       <mass value="3.1895"/>
-      <origin rpy="0.0 0.0 -1.5708" xyz="0.0001 0.0301 0.0241"/>
+      <origin rpy="0.0 0.0 -1.5708" xyz="0.0301 -0.0001 0.0241"/>
       <inertia ixx="0.0170990623" ixy="3.09e-08" ixz="-5.394e-07" iyy="0.0115476717" iyz="4.77948e-05" izz="0.0268461573"/>
     </inertial>
@@ -239,5 +239,5 @@
     <inertial>
       <mass value="0.0431"/>
-      <origin rpy="3.1416 0.0 0.0" xyz="0.0236 -0.0001 -0.003"/>
+      <origin rpy="3.1416 0.0 0.0" xyz="0.0236 0.0001 0.003"/>
       <inertia ixx="9.9689e-06" ixy="7.49e-08" ixz="-2.3932e-06" iyy="2.49545e-05" iyz="5.1e-09" izz="2.81284e-05"/>
     </inertial>
@@ -261,5 +261,5 @@
     <inertial>
       <mass value="0.0431"/>
-      <origin rpy="3.1416 0.0 0.0" xyz="0.0236 -0.0001 -0.003"/>
+      <origin rpy="3.1416 0.0 0.0" xyz="0.0236 0.0001 0.003"/>
       <inertia ixx="9.9689e-06" ixy="7.49e-08" ixz="-2.3932e-06" iyy="2.49545e-05" iyz="5.1e-09" izz="2.81284e-05"/>
     </inertial>
@@ -283,5 +283,5 @@
     <inertial>
       <mass value="0.0431"/>
-      <origin rpy="3.1416 0.0 0.0" xyz="0.0236 -0.0001 -0.003"/>
+      <origin rpy="3.1416 0.0 0.0" xyz="0.0236 0.0001 0.003"/>
       <inertia ixx="9.9689e-06" ixy="7.49e-08" ixz="-2.3932e-06" iyy="2.49545e-05" iyz="5.1e-09" izz="2.81284e-05"/>
     </inertial>
@@ -305,5 +305,5 @@
     <inertial>
       <mass value="0.0431"/>
-      <origin rpy="3.1416 0.0 0.0" xyz="0.0236 -0.0001 -0.003"/>
+      <origin rpy="3.1416 0.0 0.0" xyz="0.0236 0.0001 0.003"/>
       <inertia ixx="9.9689e-06" ixy="7.49e-08" ixz="-2.3932e-06" iyy="2.49545e-05" iyz="5.1e-09" izz="2.81284e-05"/>
     </inertial>

File: husky_description/urdf/husky_midpoint.xacro (robot description, xacro)
@@ -260,5 +260,5 @@
     <inertial>
       <mass value="3.1895"/>
-      <origin rpy="0.0 0.0 -1.5708" xyz="0.0001 0.0301 0.0241"/>
+      <origin rpy="0.0 0.0 -1.5708" xyz="0.0301 -0.0001 0.0241"/>
       <inertia ixx="0.0170990623" ixy="3.09e-08" ixz="-5.394e-07" iyy="0.0115476717" iyz="4.77948e-05" izz="0.0268461573"/>
     </inertial>
@@ -285,5 +285,5 @@
     <inertial>
       <mass value="0.0431"/>
-      <origin rpy="3.1416 0.0 0.0" xyz="0.0236 -0.0001 -0.003"/>
+      <origin rpy="3.1416 0.0 0.0" xyz="0.0236 0.0001 0.003"/>
       <inertia ixx="9.9689e-06" ixy="7.49e-08" ixz="-2.3932e-06" iyy="2.49545e-05" iyz="5.1e-09" izz="2.81284e-05"/>
     </inertial>
@@ -307,5 +307,5 @@
     <inertial>
       <mass value="0.0431"/>
-      <origin rpy="3.1416 0.0 0.0" xyz="0.0236 -0.0001 -0.003"/>
+      <origin rpy="3.1416 0.0 0.0" xyz="0.0236 0.0001 0.003"/>
       <inertia ixx="9.9689e-06" ixy="7.49e-08" ixz="-2.3932e-06" iyy="2.49545e-05" iyz="5.1e-09" izz="2.81284e-05"/>
     </inertial>
@@ -329,5 +329,5 @@
     <inertial>
       <mass value="0.0431"/>
-      <origin rpy="3.1416 0.0 0.0" xyz="0.0236 -0.0001 -0.003"/>
+      <origin rpy="3.1416 0.0 0.0" xyz="0.0236 0.0001 0.003"/>
       <inertia ixx="9.9689e-06" ixy="7.49e-08" ixz="-2.3932e-06" iyy="2.49545e-05" iyz="5.1e-09" izz="2.81284e-05"/>
     </inertial>
@@ -351,5 +351,5 @@
     <inertial>
       <mass value="0.0431"/>
-      <origin rpy="3.1416 0.0 0.0" xyz="0.0236 -0.0001 -0.003"/>
+      <origin rpy="3.1416 0.0 0.0" xyz="0.0236 0.0001 0.003"/>
       <inertia ixx="9.9689e-06" ixy="7.49e-08" ixz="-2.3932e-06" iyy="2.49545e-05" iyz="5.1e-09" izz="2.81284e-05"/>
     </inertial>

Commit message: first commit

File: husky_description/urdf/husky.xacro (robot description, xacro)
@@ -25,5 +25,5 @@
   <plugin filename="libgazebo_ros_p3d.so" name="p3d_base_controller">
     <alwaysOn>true</alwaysOn>
-    <updateRate>50.0</updateRate>
+    <updateRate>250.0</updateRate>
     <bodyName>base</bodyName>
     <topicName>ground_truth/state</topicName>
@@ -93,5 +93,5 @@
     <sensor name="imu_sensor" type="imu">
       <always_on>true</always_on>
-      <update_rate>50</update_rate>
+      <update_rate>250</update_rate>
       <visualize>true</visualize>
       <topic>__default_topic__</topic>
@@ -99,5 +99,5 @@
         <topicName>imu_link</topicName>
         <bodyName>hussain_imu</bodyName>
-        <updateRateHZ>50.0</updateRateHZ>
+        <updateRateHZ>250.0</updateRateHZ>
         <gaussianNoise>0.0</gaussianNoise>
         <xyzOffset>0 0 0</xyzOffset>
@@ -314,7 +314,7 @@
     </collision>
     <visual name="base_visual">
-      <origin rpy="0.0 0.0 -1.571" xyz="0.0 0.0 0.0"/>
-      <geometry>
-        <mesh filename="package://husky_description/meshes/body_link.STL" scale="1 1 1"/>
+      <origin rpy="-1.5708 0.0 1.5708" xyz=".212 -.258 0.128"/>
+      <geometry>
+        <mesh filename="package://husky_description/meshes/body_link_prop_part_bin.STL" scale="1 1 1"/>
       </geometry>
       <material name="">
@@ -1332,108 +1332,8 @@
 </gazebo>
 <!--ARDUCOPTER-->
-<xacro:property name="blade_x_disp" value="0.12" />
-<xacro:property name="blade_y_disp" value="0.162" />
-<!--real blades
- <link
-    name="front_right_blade">
-    <inertial>
-      <origin
-        xyz="0 0 0.004"
-        rpy="0 0 0" />
-      <mass
-        value="0.0061" />
-      <inertia ixx="9.75e-06" ixy="0" ixz="0" iyy="0.000166704" iyz="0" izz="0.000167604"/>
-    </inertial>
-  </link>
-  <link
-    name="rear_left_blade">
-    <inertial>
-      <origin
-        xyz="0 0 0.004"
-        rpy="0 0 0" />
-      <mass
-        value="0.0061" />
-      <inertia ixx="9.75e-06" ixy="0" ixz="0" iyy="0.000166704" iyz="0" izz="0.000167604"/>
-    </inertial>
-  </link>
-  <link
-    name="front_left_blade">
-    <inertial>
-      <origin
-        xyz="0 0 0.004"
-        rpy="0 0 0" />
-      <mass
-        value="0.0061" />
-      <inertia ixx="9.75e-06" ixy="0" ixz="0" iyy="0.000166704" iyz="0" izz="0.000167604"/>
-    </inertial>
-  </link>
-  <link
-    name="rear_right_blade">
-    <inertial>
-      <origin
-        xyz="0 0 0.004"
-        rpy="0 0 0" />
-      <mass
-        value="0.0061" />
-      <inertia ixx="9.75e-06" ixy="0" ixz="0" iyy="0.000166704" iyz="0" izz="0.000167604"/>
-    </inertial>
-  </link>
-  <joint
-    name="front_right_blade_joint"
-    type="revolute">
-    <origin
-      xyz="${blade_x_disp} ${-blade_y_disp} 0.062"
-      rpy="3.1416 0 0" />
-    <parent
-      link="base" />
-    <child
-      link="front_right_blade" />
-    <axis
-      xyz="0 0 1" />
-    <limit lower="-1e+16" upper="1e+16" effort="10000" velocity="10000"/>
-  </joint>
-  <joint
-    name="rear_left_blade_joint"
-    type="revolute">
-    <origin
-      xyz="${-blade_x_disp} ${blade_y_disp} 0.062"
-      rpy="0 0 0" />
-    <parent
-      link="base" />
-    <child
-      link="rear_left_blade" />
-    <axis
-      xyz="0 0 1" />
-    <limit lower="-1e+16" upper="1e+16" effort="10000" velocity="10000"/>
-  </joint>
-  <joint
-    name="front_left_blade_joint"
-    type="revolute">
-    <origin
-      xyz="${blade_x_disp} ${blade_y_disp} 0.062"
-      rpy="0 0 0" />
-    <parent
-      link="base" />
-    <child
-      link="front_left_blade" />
-    <axis
-      xyz="0 0 1" />
-    <limit lower="-1e+16" upper="1e+16" effort="10000" velocity="10000"/>
-  </joint>
-  <joint
-    name="rear_right_blade_joint"
-    type="revolute">
-    <origin
-      xyz="${-blade_x_disp} ${-blade_y_disp} 0.062"
-      rpy="3.1416 0 0" />
-    <parent
-      link="base" />
-    <child
-      link="rear_right_blade" />
-    <axis
-      xyz="0 0 1" />
-    <limit lower="-1e+16" upper="1e+16" effort="10000" velocity="10000"/>
-  </joint>
-  -->
+<xacro:property name="blade_x_disp_front" value="0.141" />
+<xacro:property name="blade_x_disp_back" value="0.125" />
+<xacro:property name="blade_y_disp" value="0.189" />
+<xacro:property name="blade_z_disp" value="0.1" />
 <!--fake blades-->
   <link
@@ -1485,5 +1385,5 @@
     type="revolute">
     <origin
-      xyz="${blade_x_disp} ${-blade_y_disp} 0.062"
+      xyz="${blade_x_disp_front} ${-blade_y_disp} ${blade_z_disp}"
       rpy="0 0 0" />
     <parent
@@ -1499,5 +1399,5 @@
     type="revolute">
     <origin
-      xyz="${blade_x_disp} ${blade_y_disp} 0.062"
+      xyz="${blade_x_disp_front} ${blade_y_disp} ${blade_z_disp}"
       rpy="0 0 0" />
     <parent
@@ -1513,5 +1413,5 @@
     type="revolute">
     <origin
-      xyz="${-blade_x_disp} ${blade_y_disp} 0.062"
+      xyz="${-blade_x_disp_back} ${blade_y_disp} ${blade_z_disp}"
       rpy="0 0 0" />
     <parent
@@ -1527,5 +1427,5 @@
     type="revolute">
     <origin
-      xyz="${-blade_x_disp} ${-blade_y_disp} 0.062"
+      xyz="${-blade_x_disp_back} ${-blade_y_disp} ${blade_z_disp}"
       rpy="0 0 0" />
     <parent
@@ -1667,4 +1567,9 @@
     <link_name>fake_rear_right_blade</link_name>
   </plugin>
+   <!--multiplier 1898, pid 0.2 0 0 -->
+  <xacro:property name="arducop_multiplier" value="1898" />
+  <xacro:property name="arducop_p" value="0.2" />
+  <xacro:property name="arducop_i" value="0" />
+  <xacro:property name="arducop_d" value="0" />
   <plugin name="arducopter_plugin" filename="libArduPilotPlugin.so">
       <fdm_addr>127.0.0.1</fdm_addr>
@@ -1689,7 +1594,7 @@
         <type>VELOCITY</type>
         <offset>0</offset>
-        <p_gain>0.2</p_gain>
-        <i_gain>0</i_gain>
-        <d_gain>0</d_gain>
+        <p_gain>${arducop_p}</p_gain>
+        <i_gain>${arducop_i}</i_gain>
+        <d_gain>${arducop_d}</d_gain>
         <i_max>0</i_max>
         <i_min>0</i_min>
@@ -1697,5 +1602,5 @@
         <cmd_min>-2.5</cmd_min>
         <jointName>fake_front_right_blade_joint</jointName>
-        <multiplier>1898</multiplier>
+        <multiplier>${arducop_multiplier}</multiplier>
         <controlVelocitySlowdownSim>1</controlVelocitySlowdownSim>
       </control>
@@ -1703,7 +1608,7 @@
         <type>VELOCITY</type>
         <offset>0</offset>
-        <p_gain>0.2</p_gain>
-        <i_gain>0</i_gain>
-        <d_gain>0</d_gain>
+        <p_gain>${arducop_p}</p_gain>
+        <i_gain>${arducop_i}</i_gain>
+        <d_gain>${arducop_d}</d_gain>
         <i_max>0</i_max>
         <i_min>0</i_min>
@@ -1711,5 +1616,5 @@
         <cmd_min>-2.5</cmd_min>
         <jointName>fake_rear_left_blade_joint</jointName>
-        <multiplier>1898</multiplier>
+        <multiplier>${arducop_multiplier}</multiplier>
         <controlVelocitySlowdownSim>1</controlVelocitySlowdownSim>
       </control>
@@ -1717,7 +1622,7 @@
         <type>VELOCITY</type>
         <offset>0</offset>
-        <p_gain>0.2</p_gain>
-        <i_gain>0</i_gain>
-        <d_gain>0</d_gain>
+        <p_gain>${arducop_p}</p_gain>
+        <i_gain>${arducop_i}</i_gain>
+        <d_gain>${arducop_d}</d_gain>
         <i_max>0</i_max>
         <i_min>0</i_min>
@@ -1725,5 +1630,5 @@
         <cmd_min>-2.5</cmd_min>
         <jointName>fake_front_left_blade_joint</jointName>
-        <multiplier>-1898</multiplier>
+        <multiplier>-${arducop_multiplier}</multiplier>
         <controlVelocitySlowdownSim>1</controlVelocitySlowdownSim>
       </control>
@@ -1731,7 +1636,7 @@
         <type>VELOCITY</type>
         <offset>0</offset>
-        <p_gain>0.2</p_gain>
-        <i_gain>0</i_gain>
-        <d_gain>0</d_gain>
+        <p_gain>${arducop_p}</p_gain>
+        <i_gain>${arducop_i}</i_gain>
+        <d_gain>${arducop_d}</d_gain>
         <i_max>0</i_max>
         <i_min>0</i_min>
@@ -1739,5 +1644,5 @@
         <cmd_min>-2.5</cmd_min>
         <jointName>fake_rear_right_blade_joint</jointName>
-        <multiplier>-1898</multiplier>
+        <multiplier>-${arducop_multiplier}</multiplier>
         <controlVelocitySlowdownSim>1</controlVelocitySlowdownSim>
       </control>

Commit message: updated keyboard

File: husky_description/urdf/husky.xacro (robot description, xacro)
@@ -142,4 +142,5 @@
     <limit effort="${efflim}" lower="${r_hip_frontal_lowlim}" upper="${r_hip_frontal_uplim}" velocity="8.7267"/>
   </joint>
+  <!--hip sag ipos -121.61 r -58.39 l-->
   <xacro:property name="fr_hip_sagittal_ipos" value="${-121.61*pi/180}" />
   <xacro:property name="fr_hip_sagittal_lowlim" value="${-12*pi/180}" />
@@ -148,4 +149,5 @@
   <xacro:property name="fl_hip_sagittal_lowlim" value="0" />
   <xacro:property name="fl_hip_sagittal_uplim" value="${12*pi/180}" />
+  <!--hip sag ipos -131.32 r -48.68 l-->
   <xacro:property name="br_hip_sagittal_ipos" value="${-131.32*pi/180}" />
   <xacro:property name="br_hip_sagittal_lowlim" value="${-12*pi/180}" />
@@ -1437,4 +1439,6 @@
     <limit lower="-1e+16" upper="1e+16" effort="10000" velocity="10000"/>
   </joint>
+<!--center of pressure, 0.084-->
+<xacro:property name="c_o_p" value="0.084" />
 <!--plugins-->
 <gazebo>
@@ -1450,5 +1454,5 @@
     <area>0.002</area>
     <air_density>1.2041</air_density>
-    <cp>0.084 0 0</cp>
+    <cp>${c_o_p} 0 0</cp>
     <forward>0 1 0</forward>
     <upward>0 0 1</upward>
@@ -1466,5 +1470,5 @@
     <area>0.002</area>
     <air_density>1.2041</air_density>
-    <cp>-0.084 0 0</cp>
+    <cp>-${c_o_p} 0 0</cp>
     <forward>0 -1 0</forward>
     <upward>0 0 1</upward>
@@ -1482,5 +1486,5 @@
     <area>0.002</area>
     <air_density>1.2041</air_density>
-    <cp>0.084 0 0</cp>
+    <cp>${c_o_p} 0 0</cp>
     <forward>0 1 0</forward>
     <upward>0 0 1</upward>
@@ -1498,5 +1502,5 @@
     <area>0.002</area>
     <air_density>1.2041</air_density>
-    <cp>-0.084 0 0</cp>
+    <cp>-${c_o_p} 0 0</cp>
     <forward>0 -1 0</forward>
     <upward>0 0 1</upward>
@@ -1514,5 +1518,5 @@
     <area>0.002</area>
     <air_density>1.2041</air_density>
-    <cp>0.084 0 0</cp>
+    <cp>${c_o_p} 0 0</cp>
     <forward>0 -1 0</forward>
     <upward>0 0 1</upward>
@@ -1530,5 +1534,5 @@
     <area>0.002</area>
     <air_density>1.2041</air_density>
-    <cp>-0.084 0 0</cp>
+    <cp>-${c_o_p} 0 0</cp>
     <forward>0 1 0</forward>
     <upward>0 0 1</upward>
@@ -1546,5 +1550,5 @@
     <area>0.002</area>
     <air_density>1.2041</air_density>
-    <cp>0.084 0 0</cp>
+    <cp>${c_o_p} 0 0</cp>
     <forward>0 -1 0</forward>
     <upward>0 0 1</upward>
@@ -1562,5 +1566,5 @@
     <area>0.002</area>
     <air_density>1.2041</air_density>
-    <cp>-0.084 0 0</cp>
+    <cp>-${c_o_p} 0 0</cp>
     <forward>0 1 0</forward>
     <upward>0 0 1</upward>
